Commit message: update vehicle scale

File: xacro/car_like_mobile_robot.xacro (robot description, xacro)
@@ -23,17 +23,18 @@
     <xacro:property name="PI" value="3.1415926535897932384626433832795028841971" />
     <!-- 車両のパラメータ -->
-    <xacro:property name="Lv" value="1.0" />
-    <xacro:property name="body_length" value="0.35" />
-    <xacro:property name="body_width" value="0.2" />
-    <xacro:property name="body_height" value="0.1" />
-    <xacro:property name="center_of_body_z" value="0.07" />
-    <!-- 骨組みのパラメータ -->
-    <xacro:property name="axel_half_length" value="${(body_width/2)*1.5}" /> <!-- 車軸半長 -->
-    <xacro:property name="axel_radius" value="0.01" /> <!-- 車軸半径 -->
-    <xacro:property name="axel_to_axel_half_length" value="0.1" /> <!-- 車軸間半長 -->
-    <xacro:property name="axel_to_axel_height" value="0.1" /> <!-- 車軸と車軸をつなぐ棒の高さ -->
+    <xacro:property name="Lv" value="1.0" /> <!-- 車軸間距離 -->
+    <xacro:property name="vehicle_body_length" value="${Lv * 1.6}" />
+    <xacro:property name="vehicle_body_width" value="${Lv * 0.8}" />
+    <xacro:property name="vehicle_body_height" value="${Lv * 0.4}" />
+    <xacro:property name="center_of_vehicle_body_z" value="${vehicle_body_height}" />
+    <xacro:property name="axel_half_length" value="${vehicle_body_width * 0.8}" /> <!-- 車軸半長 -->
+    <xacro:property name="axel_length" value="${axel_half_length * 2.0}" /> <!-- 車軸長 -->
+    <xacro:property name="axel_radius" value="0.05" /> <!-- 車軸半径 -->
+    <xacro:property name="axel_to_axel_half_length" value="${Lv * 0.5}" /> <!-- 車軸間半長 -->
+    <xacro:property name="axel_to_axel_z" value="${vehicle_body_height * 1.2}" /> <!-- 車軸と車軸をつなぐ棒の高さ -->
+    <xacro:property name="steering_length" value="${axel_to_axel_z - wheel_radius}" /> <!-- ステアリングの高さ -->
     <!-- 車輪のパラメータ -->
-    <xacro:property name="wheel_radius" value="0.05" />  <!-- 車輪半径 -->
-    <xacro:property name="wheel_width" value="0.02" />  <!-- 車輪幅 -->
+    <xacro:property name="wheel_radius" value="${Lv * 0.3}" />  <!-- 車輪半径 -->
+    <xacro:property name="wheel_width" value="${wheel_radius * 0.4}" />  <!-- 車輪幅 -->
     <xacro:property name="wheel_separation_half_length" value="${axel_half_length*0.9}" />  <!-- 車輪間半長 -->
     <!-- 車輪の回転がわかるようにするための棒のパラメータと、n番目の棒の車輪中心からの相対位置(x,y) -->
@@ -46,4 +47,33 @@
     <xacro:property name="wheel_3rd_visual_cylinder_x" value="${(wheel_radius * 2.0 / 3.0) * cos(9.0 * PI / 6.0)}" />
     <xacro:property name="wheel_3rd_visual_cylinder_y" value="${(wheel_radius * 2.0 / 3.0) * sin(9.0 * PI / 6.0)}" />
+    <!-- リンクの質量設定 -->
+    <xacro:property name="vehicle_body_mass" value="1.0" />
+    <xacro:property name="vehicle_axle_to_axel_mass" value="1.0" />
+    <xacro:property name="vehicle_steering_mass" value="1.0" />
+    <xacro:property name="vehicle_axel_mass" value="1.0" />
+    <xacro:property name="vehicle_wheel_mass" value="1.0" />
+    <xacro:property name="vehicle_wheel_visual_cylinder_mass" value="1.0" />
+    <!-- リンクのイナーシャの設定 -->
+    <xacro:property name="I_vehicle_body_xx" value="${vehicle_body_mass*(vehicle_body_height*vehicle_body_height + vehicle_body_length*vehicle_body_length) / 12}" />
+    <xacro:property name="I_vehicle_body_yy" value="${vehicle_body_mass*(vehicle_body_width*vehicle_body_width + vehicle_body_height*vehicle_body_height) / 12}" />
+    <xacro:property name="I_vehicle_body_zz" value="${vehicle_body_mass*(vehicle_body_width*vehicle_body_width + vehicle_body_length*vehicle_body_length) / 12}" />
+    <xacro:property name="I_axel_to_axel_xx" value="${vehicle_axle_to_axel_mass*Lv*Lv / 12}" />
+    <xacro:property name="I_axel_to_axel_yy" value="0.0" />
+    <xacro:property name="I_axel_to_axel_zz" value="${vehicle_axle_to_axel_mass*Lv*Lv / 12}" />
+    <xacro:property name="I_steering_xx" value="${vehicle_steering_mass*(3*axel_radius*axel_radius + steering_length*steering_length) / 12}" />
+    <xacro:property name="I_steering_yy" value="${vehicle_steering_mass*(3*axel_radius*axel_radius + steering_length*steering_length) / 12}" />
+    <xacro:property name="I_steering_zz" value="${vehicle_steering_mass*axel_radius*axel_radius / 2}" />
+    <xacro:property name="I_axel_xx" value="${vehicle_axel_mass*axel_length*axel_length / 12}" />
+    <xacro:property name="I_axel_yy" value="0.0" />
+    <xacro:property name="I_axel_zz" value="${vehicle_axel_mass*axel_length*axel_length / 12}" />
+    <xacro:property name="I_wheel_xx" value="${vehicle_wheel_mass*(3*wheel_radius*wheel_radius + wheel_width*wheel_width) / 12}" />
+    <xacro:property name="I_wheel_yy" value="${vehicle_wheel_mass*(3*wheel_radius*wheel_radius + wheel_width*wheel_width) / 12}" />
+    <xacro:property name="I_wheel_zz" value="${vehicle_wheel_mass*wheel_radius*wheel_radius / 2}" />
+    <xacro:property name="I_wheel_visual_cylinder_xx" value="${vehicle_wheel_visual_cylinder_mass*(3*wheel_visual_cylinder_radius*wheel_visual_cylinder_radius + wheel_visual_cylinder_length*wheel_visual_cylinder_length) / 12}" />
+    <xacro:property name="I_wheel_visual_cylinder_yy" value="${vehicle_wheel_visual_cylinder_mass*(3*wheel_visual_cylinder_radius*wheel_visual_cylinder_radius + wheel_visual_cylinder_length*wheel_visual_cylinder_length) / 12}" />
+    <xacro:property name="I_wheel_visual_cylinder_zz" value="${vehicle_wheel_visual_cylinder_mass*wheel_visual_cylinder_radius*wheel_visual_cylinder_radius / 2}" />
+    <!-- 摩擦力 -->
+    <xacro:property name="mu_1" value="0.5" />
+    <xacro:property name="mu_2" value="0.5" />
     <!-- 車輪の回転がわかるように埋め込む黒棒のマクロ -->
     <xacro:macro name="wheel_visual_cylinder_macro" params="vehicle front_or_rear right_or_left nth_cylinder">
@@ -64,6 +94,6 @@
             <inertial>
                 <origin xyz="0 0 0" rpy="0 0 0"/>
-                <mass value="0.1"/>
-                <inertia ixx="0.0001" ixy="0.0" ixz="0.0" iyy="0.0001" iyz="0.0" izz="0.0001"/>
+                <mass value="${vehicle_wheel_visual_cylinder_mass}"/>
+                <inertia ixx="${I_wheel_visual_cylinder_xx}" ixy="0.0" ixz="0.0" iyy="${I_wheel_visual_cylinder_yy}" iyz="0.0" izz="${I_wheel_visual_cylinder_zz}"/>
             </inertial>
             <visual>
@@ -96,10 +126,10 @@
             <inertial>
                 <origin xyz="0 0 0" rpy="0 0 0"/>
-                <mass value="0.1"/>
-                <inertia ixx="0.0001" ixy="0.0" ixz="0.0" iyy="0.0001" iyz="0.0" izz="0.0001"/>
+                <mass value="${vehicle_wheel_mass}"/>
+                <inertia ixx="${I_wheel_xx}" ixy="0.0" ixz="0.0" iyy="${I_wheel_yy}" iyz="0.0" izz="${I_wheel_zz}"/>
             </inertial>
             <visual>
                 <geometry>
-                <cylinder radius="${wheel_radius}" length="${wheel_width}" />
+                    <cylinder radius="${wheel_radius}" length="${wheel_width}" />
                 </geometry>
                 <material name="${color}"/>
@@ -107,5 +137,5 @@
             <collision>
                 <geometry>
-                <cylinder radius="${wheel_radius}" length="${wheel_width}" />
+                    <cylinder radius="${wheel_radius}" length="${wheel_width}" />
                 </geometry>
             </collision>
@@ -117,8 +147,8 @@
         <gazebo reference="${vehicle}_${front_or_rear}_${right_or_left}_link">
             <material>Gazebo/${gazebo_color}</material>
-            <!-- <mu1 value="2.5" />
-            <mu2 value="2.5" />
-            <kp value="50000" />
-            <kd value="10" /> -->
+            <mu1 value="${mu_1}" />
+            <mu2 value="${mu_2}" />
+            <kp value="500000" />
+            <kd value="10" />
         </gazebo>
     </xacro:macro>
@@ -126,19 +156,19 @@
     <link name="base_link"/>
     <!-- 胴体 -->
-    <joint name="body_joint" type="fixed">
+    <joint name="vehicle1_body_joint" type="fixed">
         <parent link="base_link"/>
-        <child  link="body_link"/>
-        <origin xyz="${axel_to_axel_half_length} 0 ${center_of_body_z}" rpy="0 0 0"/>
-    </joint>
-    <link name="body_link">
+        <child  link="vehicle1_body_link"/>
+        <origin xyz="${axel_to_axel_half_length} 0 ${center_of_vehicle_body_z}" rpy="0 0 0"/>
+    </joint>
+    <link name="vehicle1_body_link">
         <inertial>
             <origin xyz="0 0 0" rpy="0 0 0"/>
-            <mass value="1.0"/>
-            <inertia ixx="0.001" ixy="0.0" ixz="0.0" iyy="0.001" iyz="0.0" izz="0.001"/>
+            <mass value="${vehicle_body_mass}"/>
+            <inertia ixx="${I_vehicle_body_xx}" ixy="0.0" ixz="0.0" iyy="${I_vehicle_body_yy}" iyz="0.0" izz="${I_vehicle_body_zz}"/>
         </inertial>
         <visual>
             <origin xyz="0 0 0" rpy="0 0 0" />
             <geometry>
-                <box size="${body_length} ${body_width} ${body_height}" />
+                <box size="${vehicle_body_length} ${vehicle_body_width} ${vehicle_body_height}" />
             </geometry>
             <material name="gray" />
@@ -147,22 +177,22 @@
             <origin xyz="0 0 0" rpy="0 0 0" />
             <geometry>
-                <box size="${body_length} ${body_width-0.02} ${body_height}" />
-            </geometry>
-        </collision>
-    </link>
-    <gazebo reference="body_link">
+                <box size="${vehicle_body_length} ${vehicle_body_width} ${vehicle_body_height}" />
+            </geometry>
+        </collision>
+    </link>
+    <gazebo reference="vehicle1_body_link">
         <material>Gazebo/Gray</material>
     </gazebo>
     <!-- 前輪の車軸と後輪の車軸をつなぐ棒 -->
-    <joint name="axle_to_axle_joint" type="fixed">
-        <parent link="body_link"/>
-        <child  link="axel_to_axle_link"/>
-        <origin xyz="0 0 ${-center_of_body_z + axel_to_axel_height}" rpy="0 ${radians(90)} 0"/>
-    </joint>
-    <link name="axel_to_axle_link">
+    <joint name="vehicle1_axle_to_axle_joint" type="fixed">
+        <origin xyz="0 0 ${-center_of_vehicle_body_z + axel_to_axel_z}" rpy="0 ${radians(90)} 0"/>
+        <parent link="vehicle1_body_link"/>
+        <child  link="vehicle1_axel_to_axle_link"/>
+    </joint>
+    <link name="vehicle1_axel_to_axle_link">
         <inertial>
             <origin xyz="0 0 0" rpy="0 0 0"/>
-            <mass value="1.0"/>
-            <inertia ixx="0.001" ixy="0.0" ixz="0.0" iyy="0.001" iyz="0.0" izz="0.001"/>
+            <mass value="${vehicle_axle_to_axel_mass}"/>
+            <inertia ixx="${I_axel_to_axel_xx}" ixy="0.0" ixz="0.0" iyy="${I_axel_to_axel_yy}" iyz="0.0" izz="${I_axel_to_axel_zz}"/>
         </inertial>
         <visual>
@@ -180,49 +210,49 @@
         </collision>
     </link>
-    <gazebo reference="axel_to_axle_link">
+    <gazebo reference="vehicle1_axel_to_axle_link">
         <material>Gazebo/Yellow</material>
     </gazebo>
     <!-- (前輪の車軸と後輪の車軸をつなぐ棒)と(前輪の車軸)をつなぐ縦棒 -->
-    <joint name="front_steering_joint" type="revolute">
-        <parent link="axel_to_axle_link"/>
-        <child  link="front_steering_link"/>
+    <joint name="vehicle1_front_steering_joint" type="revolute">
+        <parent link="vehicle1_axel_to_axle_link"/>
+        <child  link="vehicle1_front_steering_link"/>
         <origin xyz="0 0 ${axel_to_axel_half_length}" rpy="0 ${radians(-90)} 0"/>
         <axis xyz="0 0 1" />
         <limit lower="-1.57" upper="1.57" effort="1000.0" velocity="10.0"/>
     </joint>
-    <link name="front_steering_link">
-        <inertial>
-            <origin xyz="0 0 ${-(axel_to_axel_height - wheel_radius)*0.5}" rpy="0 0 0"/>
-            <mass value="1.0"/>
-            <inertia ixx="0.001" ixy="0.0" ixz="0.0" iyy="0.001" iyz="0.0" izz="0.001"/>
-        </inertial>
-        <visual>
-        <origin xyz="0 0 ${-(axel_to_axel_height - wheel_radius)*0.5}" rpy="0 0 0" />
-            <geometry>
-                <cylinder radius="${axel_radius}" length="${axel_to_axel_height - wheel_radius}" />
-            </geometry>
-            <material name="yellow" />
-        </visual>
-        <collision>
-        <origin xyz="0 0 ${-(axel_to_axel_height - wheel_radius)*0.5}" rpy="0 0 0" />
-            <geometry>
-                <cylinder radius="${axel_radius}" length="${axel_to_axel_height - wheel_radius}" />
-            </geometry>
-        </collision>
-    </link>
-    <gazebo reference="front_steering_link">
+    <link name="vehicle1_front_steering_link">
+        <inertial>
+            <origin xyz="0 0 ${-(axel_to_axel_z - wheel_radius)*0.5}" rpy="0 0 0"/>
+            <mass value="${vehicle_steering_mass}"/>
+            <inertia ixx="${I_steering_xx}" ixy="0.0" ixz="0.0" iyy="${I_steering_yy}" iyz="0.0" izz="${I_steering_zz}"/>
+        </inertial>
+        <visual>
+        <origin xyz="0 0 ${-(axel_to_axel_z - wheel_radius)*0.5}" rpy="0 0 0" />
+            <geometry>
+                <cylinder radius="${axel_radius}" length="${axel_to_axel_z - wheel_radius}" />
+            </geometry>
+            <material name="yellow" />
+        </visual>
+        <collision>
+        <origin xyz="0 0 ${-(axel_to_axel_z - wheel_radius)*0.5}" rpy="0 0 0" />
+            <geometry>
+                <cylinder radius="${axel_radius}" length="${axel_to_axel_z - wheel_radius}" />
+            </geometry>
+        </collision>
+    </link>
+    <gazebo reference="vehicle1_front_steering_link">
         <material>Gazebo/Yellow</material>
     </gazebo>
     <!-- 前輪の車軸-->
-    <joint name="front_wheel_axle_joint" type="fixed">
-        <parent link="front_steering_link"/>
-        <child  link="front_wheel_axle_link"/>
-        <origin xyz="0 0 ${-(axel_to_axel_height - wheel_radius)}" rpy="${radians(-90)} 0 0"/>
-    </joint>
-    <link name="front_wheel_axle_link">
+    <joint name="vehicle1_front_wheel_axle_joint" type="fixed">
+        <parent link="vehicle1_front_steering_link"/>
+        <child  link="vehicle1_front_wheel_axle_link"/>
+        <origin xyz="0 0 ${-(axel_to_axel_z - wheel_radius)}" rpy="${radians(-90)} 0 0"/>
+    </joint>
+    <link name="vehicle1_front_wheel_axle_link">
         <inertial>
             <origin xyz="0 0 0" rpy="0 0 0"/>
-            <mass value="1.0"/>
-            <inertia ixx="0.001" ixy="0.0" ixz="0.0" iyy="0.001" iyz="0.0" izz="0.001"/>
+            <mass value="${vehicle_axel_mass}"/>
+            <inertia ixx="${I_axel_xx}" ixy="0.0" ixz="0.0" iyy="${I_axel_yy}" iyz="0.0" izz="${I_axel_zz}"/>
         </inertial>
         <visual>
@@ -240,50 +270,50 @@
         </collision>
     </link>
-    <gazebo reference="front_wheel_axle_link">
+    <gazebo reference="vehicle1_front_wheel_axle_link">
         <material>Gazebo/Yellow</material>
     </gazebo>
     <!-- 前輪 -->
-    <xacro:wheel_macro vehicle="vehicle1" front_or_rear="front" right_or_left="right" parent="front_wheel_axle_link" xyz="0 0 ${-wheel_separation_half_length}" color="red" gazebo_color="Red"/>
-    <xacro:wheel_macro vehicle="vehicle1" front_or_rear="front" right_or_left="left" parent="front_wheel_axle_link" xyz="0 0 ${wheel_separation_half_length}" color="red" gazebo_color="Red"/>
+    <xacro:wheel_macro vehicle="vehicle1" front_or_rear="front" right_or_left="right" parent="vehicle1_front_wheel_axle_link" xyz="0 0 ${-wheel_separation_half_length}" color="red" gazebo_color="Red"/>
+    <xacro:wheel_macro vehicle="vehicle1" front_or_rear="front" right_or_left="left" parent="vehicle1_front_wheel_axle_link" xyz="0 0 ${wheel_separation_half_length}" color="red" gazebo_color="Red"/>
     <!-- (前輪の車軸と後輪の車軸をつなぐ棒)と(後輪の車軸)をつなぐ縦棒 -->
-    <joint name="rear_steering_joint" type="fixed">
-        <parent link="axel_to_axle_link"/>
-        <child  link="rear_steering_link"/>
+    <joint name="vehicle1_rear_steering_joint" type="fixed">
         <origin xyz="0 0 ${-axel_to_axel_half_length}" rpy="0 ${radians(-90)} 0"/>
-    </joint>
-    <link name="rear_steering_link">
-        <inertial>
-            <origin xyz="0 0 ${-(axel_to_axel_height - wheel_radius)*0.5}" rpy="0 0 0"/>
-            <mass value="1.0"/>
-            <inertia ixx="0.001" ixy="0.0" ixz="0.0" iyy="0.001" iyz="0.0" izz="0.001"/>
-        </inertial>
-        <visual>
-        <origin xyz="0 0 ${-(axel_to_axel_height - wheel_radius)*0.5}" rpy="0 0 0" />
-            <geometry>
-                <cylinder radius="${axel_radius}" length="${axel_to_axel_height - wheel_radius}" />
-            </geometry>
-            <material name="yellow" />
-        </visual>
-        <collision>
-        <origin xyz="0 0 ${-(axel_to_axel_height - wheel_radius)*0.5}" rpy="0 0 0" />
-            <geometry>
-                <cylinder radius="${axel_radius}" length="${axel_to_axel_height - wheel_radius}" />
-            </geometry>
-        </collision>
-    </link>
-    <gazebo reference="rear_steering_link">
+        <parent link="vehicle1_axel_to_axle_link"/>
+        <child  link="vehicle1_rear_steering_link"/>
+    </joint>
+    <link name="vehicle1_rear_steering_link">
+        <inertial>
+            <origin xyz="0 0 ${-(steering_length)*0.5}" rpy="0 0 0"/>
+            <mass value="${vehicle_steering_mass}"/>
+            <inertia ixx="${I_steering_xx}" ixy="0.0" ixz="0.0" iyy="${I_steering_yy}" iyz="0.0" izz="${I_steering_zz}"/>
+        </inertial>
+        <visual>
+        <origin xyz="0 0 ${-(axel_to_axel_z - wheel_radius)*0.5}" rpy="0 0 0" />
+            <geometry>
+                <cylinder radius="${axel_radius}" length="${axel_to_axel_z - wheel_radius}" />
+            </geometry>
+            <material name="yellow" />
+        </visual>
+        <collision>
+        <origin xyz="0 0 ${-(axel_to_axel_z - wheel_radius)*0.5}" rpy="0 0 0" />
+            <geometry>
+                <cylinder radius="${axel_radius}" length="${axel_to_axel_z - wheel_radius}" />
+            </geometry>
+        </collision>
+    </link>
+    <gazebo reference="vehicle1_rear_steering_link">
         <material>Gazebo/Yellow</material>
     </gazebo>
     <!-- 後輪の車軸-->
-    <joint name="rear_wheel_axle_joint" type="fixed">
-        <parent link="rear_steering_link"/>
-        <child  link="rear_wheel_axle_link"/>
-        <origin xyz="0 0 ${-(axel_to_axel_height - wheel_radius)}" rpy="${radians(-90)} 0 0"/>
-    </joint>
-    <link name="rear_wheel_axle_link">
+    <joint name="vehicle1_rear_wheel_axle_joint" type="fixed">
+        <origin xyz="0 0 ${-(axel_to_axel_z - wheel_radius)}" rpy="${radians(-90)} 0 0"/>
+        <parent link="vehicle1_rear_steering_link"/>
+        <child  link="vehicle1_rear_wheel_axle_link"/>
+    </joint>
+    <link name="vehicle1_rear_wheel_axle_link">
         <inertial>
             <origin xyz="0 0 0" rpy="0 0 0"/>
-            <mass value="1.0"/>
-            <inertia ixx="0.001" ixy="0.0" ixz="0.0" iyy="0.001" iyz="0.0" izz="0.001"/>
+            <mass value="${vehicle_axel_mass}"/>
+            <inertia ixx="${I_axel_xx}" ixy="0.0" ixz="0.0" iyy="${I_axel_yy}" iyz="0.0" izz="${I_axel_zz}"/>
         </inertial>
         <visual>
@@ -301,10 +331,10 @@
         </collision>
     </link>
-    <gazebo reference="rear_wheel_axle_link">
+    <gazebo reference="vehicle1_rear_wheel_axle_link">
         <material>Gazebo/Yellow</material>
     </gazebo>
     <!-- 後輪 -->
-    <xacro:wheel_macro vehicle="vehicle1" front_or_rear="rear" right_or_left="right" parent="rear_wheel_axle_link" xyz="0 0 ${-wheel_separation_half_length}" color="blue" gazebo_color="Blue"/>
-    <xacro:wheel_macro vehicle="vehicle1" front_or_rear="rear" right_or_left="left" parent="rear_wheel_axle_link" xyz="0 0 ${wheel_separation_half_length}" color="blue" gazebo_color="Blue"/>
+    <xacro:wheel_macro vehicle="vehicle1" front_or_rear="rear" right_or_left="right" parent="vehicle1_rear_wheel_axle_link" xyz="0 0 ${-wheel_separation_half_length}" color="blue" gazebo_color="Blue"/>
+    <xacro:wheel_macro vehicle="vehicle1" front_or_rear="rear" right_or_left="left" parent="vehicle1_rear_wheel_axle_link" xyz="0 0 ${wheel_separation_half_length}" color="blue" gazebo_color="Blue"/>
     <!-- トランスミッション -->
     <!-- 前輪右車輪のトランスミッション(受動車輪のためEffort入力Effort出力) -->
@@ -349,10 +379,10 @@
     </transmission>
     <!-- 前輪ステアリングのトランスミッション(Position入力Effort出力) -->
-    <transmission name="front_steering_trans" type="SimpleTransmission">
-        <type>transmission_interface/SimpleTransmission</type>
-        <joint name="front_steering_joint">
+    <transmission name="vehicle1_front_steering_trans" type="SimpleTransmission">
+        <type>transmission_interface/SimpleTransmission</type>
+        <joint name="vehicle1_front_steering_joint">
             <hardwareInterface>hardware_interface/EffortJointInterface</hardwareInterface>
         </joint>
-        <actuator name="front_steering_motor">
+        <actuator name="vehicle1_front_steering_motor">
             <mechanicalReduction>1</mechanicalReduction>
         </actuator>
