Commit message: add lidar sensor

File: xacro/car_like_mobile_robot.xacro (robot description, xacro)
@@ -153,4 +153,64 @@
         </gazebo>
     </xacro:macro>
+    <!-- LiDARセンサのマクロ -->
+    <xacro:macro name="laser_macro" params="parent prefix xyz">
+        <joint name="${prefix}_joint" type="fixed">
+            <parent link="${parent}"/>
+            <child  link="${prefix}_link"/>
+            <origin xyz="${xyz}" rpy="0 0 0"/>
+        </joint>
+        <link name="${prefix}_link">
+            <inertial>
+                <mass value="1e-5" />
+                <origin xyz="0 0 0" rpy="0 0 0" />
+                <inertia ixx="1e-6" ixy="0" ixz="0" iyy="1e-6" iyz="0" izz="1e-6" />
+            </inertial>
+            <visual>
+                <origin xyz="0 0 0" rpy="0 0 0" />
+                <geometry>
+                    <cylinder radius="0.1" length="0.15" />
+                </geometry>
+                <material name="red" />
+            </visual>
+            <collision>
+                <origin xyz="0 0 0" rpy="0 0 0"/>
+                <geometry>
+                    <cylinder radius="0.1" length="0.15" />
+                </geometry>
+            </collision>
+        </link>
+        <gazebo reference="${prefix}_link">
+            <material>Gazebo/Red</material>
+            <sensor type="gpu_ray" name="${prefix}">
+                <pose>0 0 0 0 0 0</pose>
+                <visualize>true</visualize>
+                <update_rate>1</update_rate>
+                <ray>
+                    <scan>
+                        <horizontal>
+                            <samples>400</samples>
+                            <resolution>1</resolution>
+                            <min_angle>${-PI / 2}</min_angle>
+                            <max_angle>${PI / 2}</max_angle>
+                        </horizontal>
+                    </scan>
+                    <range>
+                        <min>0.10</min>
+                        <max>30.0</max>
+                        <resolution>0.01</resolution>
+                    </range>
+                    <noise>
+                        <type>gaussian</type>
+                        <mean>0.0</mean>
+                        <stddev>0.01</stddev>
+                    </noise>
+                </ray>
+                <plugin name="gazebo_ros_lidar_controller" filename="libgazebo_ros_gpu_laser.so">
+                    <topicName>/${prefix}_link/scan</topicName>
+                    <frameName>${prefix}_link</frameName>
+                </plugin>
+            </sensor>
+        </gazebo>
+    </xacro:macro>
     <!-- 本体 -->
     <link name="base_link"/>
@@ -184,4 +244,6 @@
         <material>Gazebo/Gray</material>
     </gazebo>
+    <!-- LiDARセンサ -->
+    <xacro:laser_macro prefix="lidar" parent="vehicle1_body_link" xyz="0 0 0.28"/>
     <!-- 前輪の車軸と後輪の車軸をつなぐ棒 -->
     <joint name="vehicle1_axle_to_axle_joint" type="fixed">

Commit message: add IMU sensor and wheel odometry and IMU integrated by ekf

File: xacro/car_like_mobile_robot.xacro (robot description, xacro)
@@ -47,4 +47,13 @@
     <xacro:property name="wheel_3rd_visual_cylinder_x" value="${(wheel_radius * 2.0 / 3.0) * cos(9.0 * PI / 6.0)}" />
     <xacro:property name="wheel_3rd_visual_cylinder_y" value="${(wheel_radius * 2.0 / 3.0) * sin(9.0 * PI / 6.0)}" />
+    <!-- LiDARセンサのパラメータ -->
+    <xacro:property name="lidar_radius" value="0.1" />
+    <xacro:property name="lidar_height" value="0.15" />
+    <xacro:property name="lidar_z" value="${center_of_vehicle_body_z + (0.5 * (vehicle_body_height + lidar_height))}" />
+    <!-- IMUセンサのパラメータ -->
+    <xacro:property name="imu_radius" value="0.08" />
+    <xacro:property name="imu_height" value="0.1" />
+    <!-- <xacro:property name="imu_z" value="${center_of_vehicle_body_z - 0.25 * vehicle_body_height}" /> -->
+    <xacro:property name="imu_z" value="${lidar_z + 0.5 * (lidar_height + imu_height)}" />
     <!-- リンクの質量設定 -->
     <xacro:property name="vehicle_body_mass" value="1.0" />
@@ -169,5 +178,5 @@
                 <origin xyz="0 0 0" rpy="0 0 0" />
                 <geometry>
-                    <cylinder radius="0.1" length="0.15" />
+                    <cylinder radius="${lidar_radius}" length="${lidar_height}" />
                 </geometry>
                 <material name="red" />
@@ -176,5 +185,5 @@
                 <origin xyz="0 0 0" rpy="0 0 0"/>
                 <geometry>
-                    <cylinder radius="0.1" length="0.15" />
+                    <cylinder radius="${lidar_radius}" length="${lidar_height}" />
                 </geometry>
             </collision>
@@ -213,4 +222,53 @@
         </gazebo>
     </xacro:macro>
+    <!-- IMUセンサを取り付けるマクロ -->
+    <xacro:macro name="imu_macro" params="parent prefix xyz">
+        <!-- IMUセンサを取り付けるジョイント -->
+        <joint name="${prefix}_joint" type="fixed">
+            <parent link="${parent}"/>
+            <child link="${prefix}_link"/>
+            <origin xyz="${xyz}" rpy="0 0 0"/>
+        </joint>
+        <!-- IMUセンサのリンク -->
+        <link name="${prefix}_link">
+            <visual>
+                <geometry>
+                    <cylinder radius="${imu_radius}" length="${imu_height}" />
+                </geometry>
+                <material name="blue"/>
+            </visual>
+            <collision>
+                <geometry>
+                    <cylinder radius="${imu_radius}" length="${imu_height}" />
+                </geometry>
+            </collision>
+            <inertial>
+                <mass value="0.01"/>
+                <inertia ixx="0.0001" ixy="0.0" ixz="0.0" iyy="0.0001" iyz="0.0" izz="0.0001"/>
+            </inertial>
+        </link>
+        <!-- Gazeboプラグインの追加 -->
+        <gazebo reference="${prefix}_link">
+            <gravity>true</gravity>
+            <material>Gazebo/Blue</material>
+            <sensor name="imu_sensor" type="imu">
+                <always_on>true</always_on>
+                <update_rate>100</update_rate>
+                <visualize>true</visualize>
+                <topic>__default_topic__</topic>
+                <plugin filename="libgazebo_ros_imu_sensor.so" name="imu_plugin">
+                    <topicName>/${prefix}_link/imu</topicName>
+                    <bodyName>${prefix}_link</bodyName>
+                    <updateRateHZ>10.0</updateRateHZ>
+                    <gaussianNoise>0.01</gaussianNoise>
+                    <xyzOffset>0 0 0</xyzOffset>
+                    <rpyOffset>0 0 0</rpyOffset>
+                    <frameName>${prefix}_link</frameName>
+                    <initialOrientationAsReference>false</initialOrientationAsReference>
+                </plugin>
+                <pose>0 0 0 0 0 0</pose>
+            </sensor>
+        </gazebo>
+    </xacro:macro>
     <!-- 本体 -->
     <link name="base_link"/>
@@ -245,5 +303,7 @@
     </gazebo>
     <!-- LiDARセンサ -->
-    <xacro:laser_macro prefix="lidar" parent="vehicle1_body_link" xyz="0 0 0.28"/>
+    <xacro:laser_macro prefix="lidar" parent="vehicle1_body_link" xyz="0 0 ${lidar_z - center_of_vehicle_body_z}"/>
+    <!-- IMUセンサ -->
+    <xacro:imu_macro prefix="imu" parent="vehicle1_body_link" xyz="0 0 ${imu_z - center_of_vehicle_body_z}"/>
     <!-- 前輪の車軸と後輪の車軸をつなぐ棒 -->
     <joint name="vehicle1_axle_to_axle_joint" type="fixed">

Commit message: adding imu filter and exec gmapping

File: xacro/car_like_mobile_robot.xacro (robot description, xacro)
@@ -54,12 +54,16 @@
     <xacro:property name="imu_radius" value="0.08" />
     <xacro:property name="imu_height" value="0.1" />
+    <!-- 車体の中に埋め込む -->
     <!-- <xacro:property name="imu_z" value="${center_of_vehicle_body_z - 0.25 * vehicle_body_height}" /> -->
+    <!-- LiDARセンサの上に乗せる -->
     <xacro:property name="imu_z" value="${lidar_z + 0.5 * (lidar_height + imu_height)}" />
+    <!-- 後輪間中点の上に乗せる -->
+    <!-- <xacro:property name="imu_z" value="${center_of_vehicle_body_z + (0.5 * (vehicle_body_height + imu_height))}" /> -->
     <!-- リンクの質量設定 -->
-    <xacro:property name="vehicle_body_mass" value="1.0" />
-    <xacro:property name="vehicle_axle_to_axel_mass" value="1.0" />
-    <xacro:property name="vehicle_steering_mass" value="1.0" />
-    <xacro:property name="vehicle_axel_mass" value="1.0" />
-    <xacro:property name="vehicle_wheel_mass" value="1.0" />
+    <xacro:property name="vehicle_body_mass" value="10.0" />
+    <xacro:property name="vehicle_axle_to_axel_mass" value="5.0" />
+    <xacro:property name="vehicle_steering_mass" value="2.5" />
+    <xacro:property name="vehicle_axel_mass" value="3.0" />
+    <xacro:property name="vehicle_wheel_mass" value="3.0" />
     <xacro:property name="vehicle_wheel_visual_cylinder_mass" value="1.0" />
     <!-- リンクのイナーシャの設定 -->
@@ -83,6 +87,8 @@
     <xacro:property name="I_wheel_visual_cylinder_zz" value="${vehicle_wheel_visual_cylinder_mass*wheel_visual_cylinder_radius*wheel_visual_cylinder_radius / 2}" />
     <!-- 摩擦力 -->
-    <xacro:property name="mu_1" value="0.5" />
-    <xacro:property name="mu_2" value="0.5" />
+    <xacro:property name="mu_1" value="0.8" />
+    <xacro:property name="mu_2" value="0.8" />
+    <xacro:property name="kp" value="500000" />
+    <xacro:property name="kd" value="10.0" />
     <!-- 車輪の回転がわかるように埋め込む黒棒のマクロ -->
     <xacro:macro name="wheel_visual_cylinder_macro" params="vehicle front_or_rear right_or_left nth_cylinder">
@@ -158,6 +164,9 @@
             <mu1 value="${mu_1}" />
             <mu2 value="${mu_2}" />
-            <kp value="500000" />
-            <kd value="10" />
+            <kp value="${kp}" />
+            <kd value="${kd}" />
+            <!-- <fdir1 value="1 0 0"/> -->
+            <!-- <minDepth value="0.001" /> -->
+            <!-- <maxContacts value="64"/> -->
         </gazebo>
     </xacro:macro>
@@ -194,9 +203,9 @@
                 <pose>0 0 0 0 0 0</pose>
                 <visualize>true</visualize>
-                <update_rate>1</update_rate>
+                <update_rate>10</update_rate>
                 <ray>
                     <scan>
                         <horizontal>
-                            <samples>400</samples>
+                            <samples>360</samples>
                             <resolution>1</resolution>
                             <min_angle>${-PI / 2}</min_angle>
@@ -257,5 +266,5 @@
                 <visualize>true</visualize>
                 <topic>__default_topic__</topic>
-                <plugin filename="libgazebo_ros_imu_sensor.so" name="imu_plugin">
+                <plugin name="imu_plugin" filename="libgazebo_ros_imu_sensor.so">
                     <topicName>/${prefix}_link/imu</topicName>
                     <bodyName>${prefix}_link</bodyName>
