Commit message: update structure of robot

File: xacro/car_like_mobile_robot.xacro (robot description, xacro)
@@ -25,17 +25,11 @@
     <xacro:property name="Lv" value="1.0" /> <!-- 車軸間距離 -->
     <xacro:property name="vehicle_body_length" value="${Lv * 1.6}" />
-    <xacro:property name="vehicle_body_width" value="${Lv * 0.8}" />
-    <xacro:property name="vehicle_body_height" value="${Lv * 0.4}" />
-    <xacro:property name="center_of_vehicle_body_z" value="${vehicle_body_height}" />
-    <xacro:property name="axel_half_length" value="${vehicle_body_width * 0.8}" /> <!-- 車軸半長 -->
-    <xacro:property name="axel_length" value="${axel_half_length * 2.0}" /> <!-- 車軸長 -->
-    <xacro:property name="axel_radius" value="0.05" /> <!-- 車軸半径 -->
-    <xacro:property name="axel_to_axel_half_length" value="${Lv * 0.5}" /> <!-- 車軸間半長 -->
-    <xacro:property name="axel_to_axel_z" value="${vehicle_body_height * 1.2}" /> <!-- 車軸と車軸をつなぐ棒の高さ -->
-    <xacro:property name="steering_length" value="${axel_to_axel_z - wheel_radius}" /> <!-- ステアリングの高さ -->
+    <xacro:property name="vehicle_body_width" value="${Lv}" />
+    <xacro:property name="vehicle_body_height" value="${Lv * 0.2}" />
+    <xacro:property name="center_of_vehicle_body_z" value="${Lv * 0.8}" />
+    <xacro:property name="wheel_base_half_length" value="${Lv * 0.5}" /> <!-- 車軸間半長 -->
     <!-- 車輪のパラメータ -->
     <xacro:property name="wheel_radius" value="${Lv * 0.3}" />  <!-- 車輪半径 -->
     <xacro:property name="wheel_width" value="${wheel_radius * 0.4}" />  <!-- 車輪幅 -->
-    <xacro:property name="wheel_separation_half_length" value="${axel_half_length*0.9}" />  <!-- 車輪間半長 -->
     <!-- 車輪の回転がわかるようにするための棒のパラメータと、n番目の棒の車輪中心からの相対位置(x,y) -->
     <xacro:property name="wheel_visual_cylinder_radius" value="${wheel_radius * 0.15}" />
@@ -47,4 +41,18 @@
     <xacro:property name="wheel_3rd_visual_cylinder_x" value="${(wheel_radius * 2.0 / 3.0) * cos(9.0 * PI / 6.0)}" />
     <xacro:property name="wheel_3rd_visual_cylinder_y" value="${(wheel_radius * 2.0 / 3.0) * sin(9.0 * PI / 6.0)}" />
+    <!-- steeringのパラメータ -->
+    <xacro:property name="steering_radius" value="${wheel_width * 0.6}" />
+    <xacro:property name="steering_height" value="${Lv * 0.04}" />
+    <xacro:property name="left_steering_y" value="${0.5*vehicle_body_width - steering_radius}" />
+    <xacro:property name="right_steering_y" value="${-0.5*vehicle_body_width + steering_radius}" />
+    <!-- steeringの下についている板とその仲間たちのパラメータ -->
+    <xacro:property name="plate_under_the_steering_length" value="${steering_radius*2.0}" />
+    <xacro:property name="plate_under_the_steering_width" value="${steering_radius*4.0}" />
+    <xacro:property name="plate_under_the_steering_height" value="${Lv * 0.04}" />
+    <xacro:property name="side_plate_of_wheel_length" value="${plate_under_the_steering_length}" />
+    <xacro:property name="side_plate_of_wheel_width" value="${0.25*(plate_under_the_steering_width-steering_radius)}" />
+    <xacro:property name="side_plate_of_wheel_height" value="${center_of_vehicle_body_z-(0.5*vehicle_body_height+steering_height+plate_under_the_steering_height) - (wheel_radius-axel_radius*2.0)}" />
+    <xacro:property name="axel_length" value="${plate_under_the_steering_width*1.05}" /> <!-- 車軸長 -->
+    <xacro:property name="axel_radius" value="0.05" /> <!-- 車軸半径 -->
     <!-- LiDARセンサのパラメータ -->
     <xacro:property name="lidar_radius" value="0.1" />
@@ -60,38 +68,58 @@
     <!-- 後輪間中点の上に乗せる -->
     <!-- <xacro:property name="imu_z" value="${center_of_vehicle_body_z + (0.5 * (vehicle_body_height + imu_height))}" /> -->
+    <!-- bodyの下に搭載する -->
+    <!-- <xacro:property name="imu_z" value="${center_of_vehicle_body_z - (0.5 * (vehicle_body_height + imu_height))}" /> -->
     <!-- リンクの質量設定 -->
-    <xacro:property name="vehicle_body_mass" value="10.0" />
-    <xacro:property name="vehicle_axle_to_axel_mass" value="5.0" />
-    <xacro:property name="vehicle_steering_mass" value="2.5" />
-    <xacro:property name="vehicle_axel_mass" value="3.0" />
-    <xacro:property name="vehicle_wheel_mass" value="3.0" />
-    <xacro:property name="vehicle_wheel_visual_cylinder_mass" value="1.0" />
+    <xacro:property name="body_mass" value="50.0" />
+    <xacro:property name="steering_mass" value="2.0" />
+    <xacro:property name="plate_under_the_steering_mass" value="2.0" />
+    <xacro:property name="side_plate_of_wheel_mass" value="8.0" />
+    <!-- 半径:0.05[m], 幅:0.288[m], 鋼の密度:7850[kg/m^3] -->
+    <xacro:property name="axel_mass" value="17.75" />
+    <!-- 外径:0.3[m], 幅:0.12[m], 内径:0.21[m], ゴムの密度:1500[kg/m^3] -->
+    <xacro:property name="wheel_mass" value="5.19" />
+    <xacro:property name="wheel_visual_cylinder_mass" value="0.0" />
+    <!-- タイヤがめり込まないように -->
+    <!-- <xacro:property name="body_mass" value="1.0" />
+    <xacro:property name="steering_mass" value="1.0" />
+    <xacro:property name="plate_under_the_steering_mass" value="1.0" />
+    <xacro:property name="side_plate_of_wheel_mass" value="1.0" />
+    <xacro:property name="axel_mass" value="5.0" />
+    <xacro:property name="wheel_mass" value="1.0" />
+    <xacro:property name="wheel_visual_cylinder_mass" value="0.0" /> -->
     <!-- リンクのイナーシャの設定 -->
-    <xacro:property name="I_vehicle_body_xx" value="${vehicle_body_mass*(vehicle_body_height*vehicle_body_height + vehicle_body_length*vehicle_body_length) / 12}" />
-    <xacro:property name="I_vehicle_body_yy" value="${vehicle_body_mass*(vehicle_body_width*vehicle_body_width + vehicle_body_height*vehicle_body_height) / 12}" />
-    <xacro:property name="I_vehicle_body_zz" value="${vehicle_body_mass*(vehicle_body_width*vehicle_body_width + vehicle_body_length*vehicle_body_length) / 12}" />
-    <xacro:property name="I_axel_to_axel_xx" value="${vehicle_axle_to_axel_mass*Lv*Lv / 12}" />
-    <xacro:property name="I_axel_to_axel_yy" value="0.0" />
-    <xacro:property name="I_axel_to_axel_zz" value="${vehicle_axle_to_axel_mass*Lv*Lv / 12}" />
-    <xacro:property name="I_steering_xx" value="${vehicle_steering_mass*(3*axel_radius*axel_radius + steering_length*steering_length) / 12}" />
-    <xacro:property name="I_steering_yy" value="${vehicle_steering_mass*(3*axel_radius*axel_radius + steering_length*steering_length) / 12}" />
-    <xacro:property name="I_steering_zz" value="${vehicle_steering_mass*axel_radius*axel_radius / 2}" />
-    <xacro:property name="I_axel_xx" value="${vehicle_axel_mass*axel_length*axel_length / 12}" />
-    <xacro:property name="I_axel_yy" value="0.0" />
-    <xacro:property name="I_axel_zz" value="${vehicle_axel_mass*axel_length*axel_length / 12}" />
-    <xacro:property name="I_wheel_xx" value="${vehicle_wheel_mass*(3*wheel_radius*wheel_radius + wheel_width*wheel_width) / 12}" />
-    <xacro:property name="I_wheel_yy" value="${vehicle_wheel_mass*(3*wheel_radius*wheel_radius + wheel_width*wheel_width) / 12}" />
-    <xacro:property name="I_wheel_zz" value="${vehicle_wheel_mass*wheel_radius*wheel_radius / 2}" />
-    <xacro:property name="I_wheel_visual_cylinder_xx" value="${vehicle_wheel_visual_cylinder_mass*(3*wheel_visual_cylinder_radius*wheel_visual_cylinder_radius + wheel_visual_cylinder_length*wheel_visual_cylinder_length) / 12}" />
-    <xacro:property name="I_wheel_visual_cylinder_yy" value="${vehicle_wheel_visual_cylinder_mass*(3*wheel_visual_cylinder_radius*wheel_visual_cylinder_radius + wheel_visual_cylinder_length*wheel_visual_cylinder_length) / 12}" />
-    <xacro:property name="I_wheel_visual_cylinder_zz" value="${vehicle_wheel_visual_cylinder_mass*wheel_visual_cylinder_radius*wheel_visual_cylinder_radius / 2}" />
+    <xacro:property name="I_body_xx" value="${body_mass*(vehicle_body_height*vehicle_body_height + vehicle_body_length*vehicle_body_length) / 12}" />
+    <xacro:property name="I_body_yy" value="${body_mass*(vehicle_body_width*vehicle_body_width + vehicle_body_height*vehicle_body_height) / 12}" />
+    <xacro:property name="I_body_zz" value="${body_mass*(vehicle_body_width*vehicle_body_width + vehicle_body_length*vehicle_body_length) / 12}" />
+    <xacro:property name="I_steering_xx" value="${steering_mass*(3*axel_radius*axel_radius + steering_height*steering_height) / 12}" />
+    <xacro:property name="I_steering_yy" value="${steering_mass*(3*axel_radius*axel_radius + steering_height*steering_height) / 12}" />
+    <xacro:property name="I_steering_zz" value="${steering_mass*axel_radius*axel_radius / 2}" />
+    <xacro:property name="I_plate_under_the_steering_xx" value="${plate_under_the_steering_mass*(plate_under_the_steering_height*plate_under_the_steering_height + plate_under_the_steering_length*plate_under_the_steering_length) / 12}" />
+    <xacro:property name="I_plate_under_the_steering_yy" value="${plate_under_the_steering_mass*(plate_under_the_steering_width*plate_under_the_steering_width + plate_under_the_steering_height*plate_under_the_steering_height) / 12}" />
+    <xacro:property name="I_plate_under_the_steering_zz" value="${plate_under_the_steering_mass*(plate_under_the_steering_width*plate_under_the_steering_width + plate_under_the_steering_length*plate_under_the_steering_length) / 12}" />
+    <xacro:property name="I_side_plate_of_wheel_xx" value="${side_plate_of_wheel_mass*(side_plate_of_wheel_height*side_plate_of_wheel_height + side_plate_of_wheel_length*side_plate_of_wheel_length) / 12}" />
+    <xacro:property name="I_side_plate_of_wheel_yy" value="${side_plate_of_wheel_mass*(side_plate_of_wheel_width*side_plate_of_wheel_width + side_plate_of_wheel_height*side_plate_of_wheel_height) / 12}" />
+    <xacro:property name="I_side_plate_of_wheel_zz" value="${side_plate_of_wheel_mass*(side_plate_of_wheel_width*side_plate_of_wheel_width + side_plate_of_wheel_length*side_plate_of_wheel_length) / 12}" />
+    <xacro:property name="I_axel_xx" value="${axel_mass*(3*axel_radius*axel_radius + axel_length*axel_length) / 12}" />
+    <xacro:property name="I_axel_yy" value="${axel_mass*(3*axel_radius*axel_radius + axel_length*axel_length) / 12}" />
+    <xacro:property name="I_axel_zz" value="${axel_mass*axel_radius*axel_radius / 2}" />
+    <xacro:property name="I_wheel_xx" value="${wheel_mass*(3*wheel_radius*wheel_radius + wheel_width*wheel_width) / 12}" />
+    <xacro:property name="I_wheel_yy" value="${wheel_mass*(3*wheel_radius*wheel_radius + wheel_width*wheel_width) / 12}" />
+    <xacro:property name="I_wheel_zz" value="${wheel_mass*wheel_radius*wheel_radius / 2}" />
+    <xacro:property name="I_wheel_visual_cylinder_xx" value="${wheel_visual_cylinder_mass*(3*wheel_visual_cylinder_radius*wheel_visual_cylinder_radius + wheel_visual_cylinder_length*wheel_visual_cylinder_length) / 12}" />
+    <xacro:property name="I_wheel_visual_cylinder_yy" value="${wheel_visual_cylinder_mass*(3*wheel_visual_cylinder_radius*wheel_visual_cylinder_radius + wheel_visual_cylinder_length*wheel_visual_cylinder_length) / 12}" />
+    <xacro:property name="I_wheel_visual_cylinder_zz" value="${wheel_visual_cylinder_mass*wheel_visual_cylinder_radius*wheel_visual_cylinder_radius / 2}" />
     <!-- 摩擦力 -->
-    <xacro:property name="mu_1" value="0.8" />
-    <xacro:property name="mu_2" value="0.8" />
-    <xacro:property name="kp" value="500000" />
-    <xacro:property name="kd" value="10.0" />
+    <!-- <xacro:property name="mu_1" value="0.8" />
+    <xacro:property name="mu_2" value="0.8" /> -->
+    <xacro:property name="mu_1" value="1.2" />
+    <xacro:property name="mu_2" value="1.2" />
+    <!-- <xacro:property name="mu_1" value="10" />
+    <xacro:property name="mu_2" value="10" /> -->
+    <xacro:property name="kp" value="2000000" />
+    <xacro:property name="kd" value="100" />
     <!-- 車輪の回転がわかるように埋め込む黒棒のマクロ -->
-    <xacro:macro name="wheel_visual_cylinder_macro" params="vehicle front_or_rear right_or_left nth_cylinder">
-        <joint name="${vehicle}_${front_or_rear}_${right_or_left}_${nth_cylinder}_joint" type="fixed">
+    <xacro:macro name="wheel_visual_cylinder_macro" params="vehicle front_or_rear left_or_right nth_cylinder">
+        <joint name="${vehicle}_${front_or_rear}_${left_or_right}_${nth_cylinder}_joint" type="fixed">
             <xacro:if value="${nth_cylinder=='first'}">
                 <origin xyz="${wheel_1st_visual_cylinder_x} ${wheel_1st_visual_cylinder_y} 0" rpy="0 0 0"/>
@@ -103,16 +131,16 @@
                 <origin xyz="${wheel_3rd_visual_cylinder_x} ${wheel_3rd_visual_cylinder_y} 0" rpy="0 0 0"/>
             </xacro:if>
-            <parent link="${vehicle}_${front_or_rear}_${right_or_left}_link"/>
-            <child  link="${vehicle}_${front_or_rear}_${right_or_left}_${nth_cylinder}_link"/>
-        </joint>
-        <link name="${vehicle}_${front_or_rear}_${right_or_left}_${nth_cylinder}_link">
-            <inertial>
-                <origin xyz="0 0 0" rpy="0 0 0"/>
-                <mass value="${vehicle_wheel_visual_cylinder_mass}"/>
+            <parent link="${vehicle}_${front_or_rear}_${left_or_right}_link"/>
+            <child  link="${vehicle}_${front_or_rear}_${left_or_right}_${nth_cylinder}_link"/>
+        </joint>
+        <link name="${vehicle}_${front_or_rear}_${left_or_right}_${nth_cylinder}_link">
+            <inertial>
+                <origin xyz="0 0 0" rpy="0 0 0"/>
+                <mass value="${wheel_visual_cylinder_mass}"/>
                 <inertia ixx="${I_wheel_visual_cylinder_xx}" ixy="0.0" ixz="0.0" iyy="${I_wheel_visual_cylinder_yy}" iyz="0.0" izz="${I_wheel_visual_cylinder_zz}"/>
             </inertial>
             <visual>
                 <geometry>
-                <cylinder radius="${wheel_visual_cylinder_radius}" length="${wheel_visual_cylinder_length}" />
+                    <cylinder radius="${wheel_visual_cylinder_radius}" length="${wheel_visual_cylinder_length}" />
                 </geometry>
                 <material name="black"/>
@@ -120,26 +148,26 @@
             <collision>
                 <geometry>
-                <cylinder radius="${wheel_visual_cylinder_radius}" length="${wheel_visual_cylinder_length}" />
-                </geometry>
-            </collision>
-        </link>
-        <gazebo reference="${vehicle}_${front_or_rear}_${right_or_left}_${nth_cylinder}_link">
+                    <cylinder radius="${wheel_visual_cylinder_radius}" length="${wheel_visual_cylinder_length}" />
+                </geometry>
+            </collision>
+        </link>
+        <gazebo reference="${vehicle}_${front_or_rear}_${left_or_right}_${nth_cylinder}_link">
             <material>Gazebo/Black</material>
         </gazebo>
     </xacro:macro>
-    <!-- 車輪のマクロ -->
-    <xacro:macro name="wheel_macro" params="parent vehicle front_or_rear right_or_left xyz color gazebo_color">
-        <joint name="${vehicle}_${front_or_rear}_${right_or_left}_joint" type="continuous">
-            <origin xyz="${xyz}" rpy="0 0 0"/>
+    <!-- wheel macro -->
+    <xacro:macro name="wheel_macro" params="parent vehicle front_or_rear left_or_right color gazebo_color">
+        <joint name="${vehicle}_${front_or_rear}_${left_or_right}_joint" type="continuous">
+            <origin xyz="0 0 ${-(center_of_vehicle_body_z - 0.5*(vehicle_body_height +steering_height) - wheel_radius)}" rpy="${radians(-90)} 0 0"/>
             <parent link="${parent}"/>
-            <child  link="${vehicle}_${front_or_rear}_${right_or_left}_link"/>
+            <child  link="${vehicle}_${front_or_rear}_${left_or_right}_link"/>
             <axis xyz="0 0 1" />
-            <!-- <limit velocity="12.0" effort="10.0" /> -->
+            <limit velocity="10.0" effort="51.0" />
             <!-- <dynamics damping="0.1"/> -->
         </joint>
-        <link name="${vehicle}_${front_or_rear}_${right_or_left}_link">
-            <inertial>
-                <origin xyz="0 0 0" rpy="0 0 0"/>
-                <mass value="${vehicle_wheel_mass}"/>
+        <link name="${vehicle}_${front_or_rear}_${left_or_right}_link">
+            <inertial>
+                <origin xyz="0 0 0" rpy="0 0 0"/>
+                <mass value="${wheel_mass}"/>
                 <inertia ixx="${I_wheel_xx}" ixy="0.0" ixz="0.0" iyy="${I_wheel_yy}" iyz="0.0" izz="${I_wheel_zz}"/>
             </inertial>
@@ -157,8 +185,8 @@
         </link>
         <!-- 回転がわかるように3つの黒棒を埋め込む -->
-        <xacro:wheel_visual_cylinder_macro vehicle="${vehicle}" front_or_rear="${front_or_rear}" right_or_left="${right_or_left}" nth_cylinder="first"/>
-        <xacro:wheel_visual_cylinder_macro vehicle="${vehicle}" front_or_rear="${front_or_rear}" right_or_left="${right_or_left}" nth_cylinder="second"/>
-        <xacro:wheel_visual_cylinder_macro vehicle="${vehicle}" front_or_rear="${front_or_rear}" right_or_left="${right_or_left}" nth_cylinder="third"/>
-        <gazebo reference="${vehicle}_${front_or_rear}_${right_or_left}_link">
+        <xacro:wheel_visual_cylinder_macro vehicle="${vehicle}" front_or_rear="${front_or_rear}" left_or_right ="${left_or_right}" nth_cylinder="first"/>
+        <xacro:wheel_visual_cylinder_macro vehicle="${vehicle}" front_or_rear="${front_or_rear}" left_or_right ="${left_or_right}" nth_cylinder="second"/>
+        <xacro:wheel_visual_cylinder_macro vehicle="${vehicle}" front_or_rear="${front_or_rear}" left_or_right ="${left_or_right}" nth_cylinder="third"/>
+        <gazebo reference="${vehicle}_${front_or_rear}_${left_or_right}_link">
             <material>Gazebo/${gazebo_color}</material>
             <mu1 value="${mu_1}" />
@@ -171,4 +199,150 @@
         </gazebo>
     </xacro:macro>
+    <!-- side_plate_of_wheel_macro -->
+    <xacro:macro name="side_plate_of_wheel_macro" params="parent front_or_rear left_or_right left_plate_or_right_plate">
+        <joint name="vehicle1_${left_plate_or_right_plate}_plate_of_${front_or_rear}_${left_or_right}_wheel_joint" type="fixed">
+            <xacro:if value="${left_plate_or_right_plate=='left'}">
+                <origin xyz="0 ${0.5*(plate_under_the_steering_width - side_plate_of_wheel_width)} ${-0.5 *(plate_under_the_steering_height + side_plate_of_wheel_height)}" rpy="0 0 0"/>
+            </xacro:if>
+            <xacro:if value="${left_plate_or_right_plate=='right'}">
+                <origin xyz="0 ${-0.5*(plate_under_the_steering_width - side_plate_of_wheel_width)} ${-0.5 *(plate_under_the_steering_height + side_plate_of_wheel_height)}" rpy="0 0 0"/>
+            </xacro:if>
+            <parent link="${parent}"/>
+            <child  link="vehicle1_${left_plate_or_right_plate}_plate_of_${front_or_rear}_${left_or_right}_wheel_link"/>
+        </joint>
+        <link name="vehicle1_${left_plate_or_right_plate}_plate_of_${front_or_rear}_${left_or_right}_wheel_link">
+            <inertial>
+                <origin xyz="0 0 0" rpy="0 0 0"/>
+                <mass value="${side_plate_of_wheel_mass}"/>
+                <inertia ixx="${I_side_plate_of_wheel_xx}" ixy="0.0" ixz="0.0" iyy="${I_side_plate_of_wheel_yy}" iyz="0.0" izz="${I_side_plate_of_wheel_zz}"/>
+            </inertial>
+            <visual>
+            <origin xyz="0 0 0" rpy="0 0 0" />
+                <geometry>
+                    <box size="${side_plate_of_wheel_length} ${side_plate_of_wheel_width} ${side_plate_of_wheel_height}" />
+                </geometry>
+                <material name="yellow" />
+            </visual>
+            <collision>
+            <origin xyz="0 0 0" rpy="0 0 0" />
+                <geometry>
+                    <box size="${side_plate_of_wheel_length} ${side_plate_of_wheel_width} ${side_plate_of_wheel_height}" />
+                </geometry>
+            </collision>
+        </link>
+        <gazebo reference="vehicle1_${left_plate_or_right_plate}_plate_of_${front_or_rear}_${left_or_right}_wheel_link">
+            <material>Gazebo/Yellow</material>
+        </gazebo>
+    </xacro:macro>
+    <!-- ${front_or_rear}_${left_or_right}_steering_and_wheel_macro -->
+    <xacro:macro name="steering_and_wheel_macro" params="parent xyz front_or_rear left_or_right">
+        <!-- steering -->
+        <xacro:if value="${front_or_rear=='front'}">
+            <xacro:property name="wheel_joint_type" value="revolute" />
+        </xacro:if>
+        <xacro:if value="${front_or_rear=='rear'}">
+            <xacro:property name="wheel_joint_type" value="fixed" />
+        </xacro:if>
+        <joint name="vehicle1_${front_or_rear}_${left_or_right}_steering_joint" type="${wheel_joint_type}">
+            <origin xyz="${xyz}" rpy="0 0 0"/>
+            <parent link="${parent}"/>
+            <child  link="vehicle1_${front_or_rear}_${left_or_right}_steering_link"/>
+            <xacro:if value="${front_or_rear=='front'}">
+                <axis xyz="0 0 1" />
+                <limit lower="-1.57" upper="1.57" effort="1000.0" velocity="10.0"/>
+            </xacro:if>
+        </joint>
+        <link name="vehicle1_${front_or_rear}_${left_or_right}_steering_link">
+            <inertial>
+                <origin xyz="0 0 0" rpy="0 0 0"/>
+                <mass value="${steering_mass}"/>
+                <inertia ixx="${I_steering_xx}" ixy="0.0" ixz="0.0" iyy="${I_steering_yy}" iyz="0.0" izz="${I_steering_zz}"/>
+            </inertial>
+            <visual>
+            <origin xyz="0 0 0" rpy="0 0 0" />
+                <geometry>
+                    <cylinder radius="${steering_radius}" length="${steering_height}" />
+                </geometry>
+                <material name="yellow" />
+            </visual>
+            <collision>
+            <origin xyz="0 0 0" rpy="0 0 0" />
+                <geometry>
+                    <cylinder radius="${steering_radius}" length="${steering_height}" />
+                </geometry>
+            </collision>
+        </link>
+        <gazebo reference="vehicle1_${front_or_rear}_${left_or_right}_steering_link">
+            <material>Gazebo/Yellow</material>
+        </gazebo>
+        <!-- wheel -->
+        <xacro:if value="${front_or_rear=='front'}">
+            <xacro:wheel_macro vehicle="vehicle1" front_or_rear="${front_or_rear}" left_or_right ="${left_or_right}" parent="vehicle1_${front_or_rear}_${left_or_right}_steering_link" color="red" gazebo_color="Red"/>
+        </xacro:if>
+        <xacro:if value="${front_or_rear=='rear'}">
+            <xacro:wheel_macro vehicle="vehicle1" front_or_rear="${front_or_rear}" left_or_right ="${left_or_right}" parent="vehicle1_${front_or_rear}_${left_or_right}_steering_link" color="blue" gazebo_color="Blue"/>
+        </xacro:if>
+        <!-- plate under the steering -->
+        <joint name="vehicle1_plate_under_the_${front_or_rear}_${left_or_right}_steering_joint" type="fixed">
+            <origin xyz="0 0 ${-0.5 *(steering_height + plate_under_the_steering_height)}" rpy="0 0 0"/>
+            <parent link="vehicle1_${front_or_rear}_${left_or_right}_steering_link"/>
+            <child  link="vehicle1_plate_under_the_${front_or_rear}_${left_or_right}_steering_link"/>
+        </joint>
+        <link name="vehicle1_plate_under_the_${front_or_rear}_${left_or_right}_steering_link">
+            <inertial>
+                <origin xyz="0 0 0" rpy="0 0 0"/>
+                <mass value="${plate_under_the_steering_mass}"/>
+                <inertia ixx="${I_plate_under_the_steering_xx}" ixy="0.0" ixz="0.0" iyy="${I_plate_under_the_steering_yy}" iyz="0.0" izz="${I_plate_under_the_steering_zz}"/>
+            </inertial>
+            <visual>
+            <origin xyz="0 0 0" rpy="0 0 0" />
+                <geometry>
+                    <box size="${plate_under_the_steering_length} ${plate_under_the_steering_width} ${plate_under_the_steering_height}" />
+                </geometry>
+                <material name="yellow" />
+            </visual>
+            <collision>
+            <origin xyz="0 0 0" rpy="0 0 0" />
+                <geometry>
+                    <box size="${plate_under_the_steering_length} ${plate_under_the_steering_width} ${plate_under_the_steering_height}" />
+                </geometry>
+            </collision>
+        </link>
+        <gazebo reference="vehicle1_plate_under_the_${front_or_rear}_${left_or_right}_steering_link">
+            <material>Gazebo/Yellow</material>
+        </gazebo>
+        <!-- side plate of wheel -->
+        <xacro:side_plate_of_wheel_macro parent="vehicle1_plate_under_the_${front_or_rear}_${left_or_right}_steering_link" front_or_rear="${front_or_rear}" left_or_right="${left_or_right}" left_plate_or_right_plate="left"/>
+        <xacro:side_plate_of_wheel_macro parent="vehicle1_plate_under_the_${front_or_rear}_${left_or_right}_steering_link" front_or_rear="${front_or_rear}" left_or_right="${left_or_right}" left_plate_or_right_plate="right"/>
+        <!-- axel of wheel -->
+        <joint name="vehicle1_${front_or_rear}_${left_or_right}_wheel_axle_joint" type="fixed">
+            <origin xyz="0 0 ${-((center_of_vehicle_body_z - 0.5*vehicle_body_height -steering_height -0.5*plate_under_the_steering_height) - wheel_radius)}" rpy="${radians(-90)} 0 0"/>
+            <parent link="vehicle1_plate_under_the_${front_or_rear}_${left_or_right}_steering_link"/>
+            <child  link="vehicle1_${front_or_rear}_${left_or_right}_wheel_axle_link"/>
+        </joint>
+        <link name="vehicle1_${front_or_rear}_${left_or_right}_wheel_axle_link">
+            <inertial>
+                <origin xyz="0 0 0" rpy="0 0 0"/>
+                <mass value="${axel_mass}"/>
+                <inertia ixx="${I_axel_xx}" ixy="0.0" ixz="0.0" iyy="${I_axel_yy}" iyz="0.0" izz="${I_axel_zz}"/>
+            </inertial>
+            <visual>
+            <origin xyz="0 0 0" rpy="0 0 0" />
+                <geometry>
+                    <cylinder radius="${axel_radius}" length="${axel_length}" />
+                </geometry>
+                <material name="black" />
+            </visual>
+            <collision>
+            <origin xyz="0 0 0" rpy="0 0 0" />
+                <geometry>
+                    <cylinder radius="${axel_radius}" length="${axel_length}" />
+                </geometry>
+            </collision>
+        </link>
+        <gazebo reference="vehicle1_${front_or_rear}_${left_or_right}_wheel_axle_link">
+            <material>Gazebo/Black</material>
+        </gazebo>
+    </xacro:macro>
     <!-- LiDARセンサのマクロ -->
     <xacro:macro name="laser_macro" params="parent prefix xyz">
@@ -202,10 +376,10 @@
             <sensor type="gpu_ray" name="${prefix}">
                 <pose>0 0 0 0 0 0</pose>
-                <visualize>true</visualize>
-                <update_rate>10</update_rate>
+                <visualize>false</visualize>
+                <update_rate>30</update_rate>
                 <ray>
                     <scan>
                         <horizontal>
-                            <samples>360</samples>
+                            <samples>720</samples>
                             <resolution>1</resolution>
                             <min_angle>${-PI / 2}</min_angle>
@@ -221,5 +395,5 @@
                         <type>gaussian</type>
                         <mean>0.0</mean>
-                        <stddev>0.01</stddev>
+                        <stddev>0.001</stddev>
                     </noise>
                 </ray>
@@ -263,5 +437,5 @@
             <sensor name="imu_sensor" type="imu">
                 <always_on>true</always_on>
-                <update_rate>100</update_rate>
+                <update_rate>1000</update_rate>
                 <visualize>true</visualize>
                 <topic>__default_topic__</topic>
@@ -271,8 +445,9 @@
                     <updateRateHZ>10.0</updateRateHZ>
                     <gaussianNoise>0.01</gaussianNoise>
+                    <!-- <gaussianNoise>0.00</gaussianNoise> -->
                     <xyzOffset>0 0 0</xyzOffset>
                     <rpyOffset>0 0 0</rpyOffset>
                     <frameName>${prefix}_link</frameName>
-                    <initialOrientationAsReference>false</initialOrientationAsReference>
+                    <!-- <initialOrientationAsReference>false</initialOrientationAsReference> -->
                 </plugin>
                 <pose>0 0 0 0 0 0</pose>
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